File: battery-board.kicad_pcb (KiCad board)
At the start: 4 copper layers, 84.8 x 100 mm, 203 parts, among them J1 JST-XH, J10 XT60-M, J11 XT60-F, J12 XT60-F, J13 XT60-F, J14 XT60-F, J15 XT60-F, J16 XT60-F, J17 XT60-F, J18 XT60-F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

Commit message: gerber output
Routing:
- net BATTP_CHG: track 25.9 -> 22.2 mm
- net /load_switch/DSG_GATE: track 40.2 -> 38.8 mm, vias 3 -> 2
- net BATTN: track 282.5 -> 281.3 mm, vias 110 -> 107
- net VCHG_SENSE: track 121.6 -> 121.0 mm
- net /load_switch/CHG_SRC: track 58.4 -> 59.0 mm
Other:
- rule pad_to_mask_clearance: 0.05 -> 0.1
