File: power_connectors.kicad_sch (KiCad schematic)
At the start: 21 parts, among them J10 XT60-M, J11 XT60-F, J12 XT60-F, J13 XT60-F, J14 XT60-F, J15 XT60-F, J16 XT60-F, J17 XT60-F, J18 XT60-F, J9 XT60-M

Commit message: gerber output
Changed lines of the file:
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@@
   (junction (at 77.47 165.1) (diameter 0) (color 0 0 0 0)
   )
-  (junction (at 41.91 24.13) (diameter 0) (color 0 0 0 0)
-  )
   (junction (at 62.23 125.73) (diameter 0) (color 0 0 0 0)
   )
@@
     (stroke (width 0) (type default) (color 0 0 0 0))
   )
-  (wire (pts (xy 38.1 24.13) (xy 41.91 24.13))
-    (stroke (width 0) (type default) (color 0 0 0 0))
-  )
   (wire (pts (xy 63.5 72.39) (xy 90.17 72.39))
     (stroke (width 0) (type default) (color 0 0 0 0))
@@
     (stroke (width 0) (type default) (color 0 0 0 0))
   )
-  (wire (pts (xy 41.91 24.13) (xy 41.91 26.67))
-    (stroke (width 0) (type default) (color 0 0 0 0))
-  )
   (wire (pts (xy 63.5 27.94) (xy 90.17 27.94))
     (stroke (width 0) (type default) (color 0 0 0 0))
@@
     (stroke (width 0) (type default) (color 0 0 0 0))
   )
-  (wire (pts (xy 41.91 24.13) (xy 53.34 24.13))
+  (wire (pts (xy 38.1 24.13) (xy 53.34 24.13))
     (stroke (width 0) (type default) (color 0 0 0 0))
   )
@@
   )
   (wire (pts (xy 63.5 163.83) (xy 63.5 165.1))
-    (stroke (width 0) (type default) (color 0 0 0 0))
-  )
-  (wire (pts (xy 41.91 34.29) (xy 41.91 36.83))
     (stroke (width 0) (type default) (color 0 0 0 0))
   )
@@
     (pin "2")
   )
-  (symbol (lib_id "power:GNDPWR") (at 41.91 36.83 0) (unit 1)
-    (in_bom yes) (on_board yes) (fields_autoplaced)
-    (property "Reference" "#PWR0114" (id 0) (at 41.91 41.91 0)
-      (effects (font (size 1.27 1.27)) hide)
-    )
-    (property "Value" "GNDPWR" (id 1) (at 41.783 41.91 0))
-    (property "Footprint" "" (id 2) (at 41.91 38.1 0)
-      (effects (font (size 1.27 1.27)) hide)
-    )
-    (property "Datasheet" "" (id 3) (at 41.91 38.1 0)
-      (effects (font (size 1.27 1.27)) hide)
-    )
-    (pin "1")
-  )
   (symbol (lib_id "Connector:Conn_01x02_Female") (at 95.25 69.85 0) (unit 1)
